Commit message: add gripper

File: urdf/base/base.gazebo.xacro (robot description, xacro)
@@ -6,5 +6,5 @@
       </gazebo>
       <gazebo reference="base_link">
-          <gravity>false</gravity>
+          <gravity>true</gravity>
           <material value="Gazebo/Grey"/>
       </gazebo>
@@ -12,6 +12,6 @@
       <gazebo reference="wheel_left_link">
           <gravity>true</gravity>
-          <mu1>1.5</mu1>
-          <mu2>1.5</mu2>
+          <mu1>100.5</mu1>
+          <mu2>100.5</mu2>
           <kp>1000000.0</kp>
           <kd>100.0</kd>
@@ -22,6 +22,6 @@
       <gazebo reference="wheel_right_link">
           <gravity>true</gravity>
-          <mu1>1.5</mu1>
-          <mu2>1.5</mu2>
+          <mu1>100.5</mu1>
+          <mu2>100.5</mu2>
           <kp>1000000.0</kp>
           <kd>100.0</kd>
@@ -32,15 +32,17 @@
       <gazebo reference="hanger">
           <gravity>true</gravity>
-          <mu1>0.0</mu1>
-          <mu2>0.0</mu2>
-          <material value="Gazebo/Grey"/>
-      </gazebo>
-      <gazebo reference="castor_front">
-          <gravity>true</gravity>
-          <mu1>0.0</mu1>
-          <mu2>0.0</mu2>
+          <mu1>0.1</mu1>
+          <mu2>0.1</mu2>
           <kp>1000000.0</kp>
           <kd>100.0</kd>
           <material value="Gazebo/Grey"/>
       </gazebo>
+      <!--<gazebo reference="castor_front">
+          <gravity>true</gravity>
+          <mu1>0.1</mu1>
+          <mu2>0.1</mu2>
+          <kp>1000000.0</kp>
+          <kd>100.0</kd>
+          <material value="Gazebo/Grey"/>
+      </gazebo>-->
 </robot>

File: urdf/base/base_mp500.urdf.xacro (robot description, xacro)
@@ -18,7 +18,8 @@
 	<link name="base_link">
 		<inertial>
-			<mass value="25.67" />
-			<origin xyz="0 0 0.216" rpy="0 0 0"/>
-			<inertia ixx="0.54" ixy="0.0" ixz="0.0" iyy="1.08" iyz="0.0" izz="1.23" />
+			<mass value="1" />
+			<!--<origin xyz="0 0 0.216" rpy="0 0 0"/>-->
+			<!--<inertia ixx="0.54" ixy="0.0" ixz="0.0" iyy="1.08" iyz="0.0" izz="1.23" />-->
+			<inertia ixx="1" ixy="0.0" ixz="0.0" iyy="1" iyz="0.0" izz="1" />
 		</inertial>
 		<visual name='body'>
@@ -67,5 +68,5 @@
 		<origin xyz="-0.155 0.255 0.13" rpy="0 0 0" />
 		<axis xyz="0 1 0"/>
-		<limit effort="20" velocity="1.5"/>
+		<limit effort="500" velocity="5"/>
 		<dynamics damping="0.0" friction="0.0" />
 		<parent link="base_link" />
@@ -126,5 +127,5 @@
 		<origin xyz="-0.155 -0.255 0.13" rpy="0 0 0" />
 		<axis xyz="0 1 0"/>
-		<limit effort="20" velocity="1.5"/>
+		<limit effort="500" velocity="5"/>
 		<dynamics damping="0.0" friction="0.0" />
 		<parent link="base_link" />
@@ -148,5 +149,5 @@
 			<origin xyz="0 0 0" rpy="0 0 -1.57" />
 			<geometry>
-				<sphere radius="0.00115"/>
+				<mesh filename="package://mp500lwa4d_description/meshes/mp500/HANGER-WHEEL.STL" scale="0.01 0.01 0.01" />
 			</geometry>
 		</collision>
@@ -158,30 +159,3 @@
 		<child link="hanger" />
 	</joint>
-<!--+++++++++++++++ castor_front +++++++++++++++-->
-	<link name="castor_front">
-		<inertial>
-			<mass value="0.001" />
-			<origin xyz="0 0 0" rpy="0 0 0" />
-			<inertia ixx="0.000025" ixy="0" ixz="0" iyy="0.000025" iyz="0" izz="0.000025" />
-		</inertial>
-		<visual>
-			<origin xyz="0 0 0" rpy="0 0 0" />
-			<geometry>
-				<sphere radius="0.005"/>
-			</geometry>
-			<material name="Grey" />
-		</visual>
-		<collision>
-			<origin xyz="0 0 0" rpy="0 0 0" />
-			<geometry>
-				<sphere radius="0.005"/>
-			</geometry>
-		</collision>
-	</link>
-	<joint name="castor_front_joint" type="fixed">
-		<origin xyz="0.3 0 0.01" rpy="0 0 0"/>
-		<axis xyz="0 0 1"/>
-		<parent link="base_link" />
-		<child link="castor_front" />
-	</joint>
 </robot>

File: urdf/robot.gazebo.xacro (robot description, xacro)
@@ -2,4 +2,8 @@
 <robot xmlns:xacro="http://www.ros.org/wiki/xacro">
     <gazebo>
+        <plugin name="gazebo_ros_control" filename="libgazebo_ros_control.so">
+            <robotNamespace>/mp500lwa4d</robotNamespace>
+            <robotBaseFrame>base_footprint</robotBaseFrame>
+        </plugin>
         <plugin name="differential_drive_controller" filename="libgazebo_ros_diff_drive.so">
         <robotNamespace>/mp500lwa4d</robotNamespace>
@@ -10,5 +14,5 @@
         <wheelSeparation>0.51</wheelSeparation>
         <wheelDiameter>0.25</wheelDiameter>
-        <torque>30</torque>
+        <torque>100</torque>
         <commandTopic>/mobile_base_controller/cmd_vel</commandTopic>
         <odometryTopic>odom</odometryTopic>
@@ -19,14 +23,10 @@
         <publishWheelTF>true</publishWheelTF>
         <publishWheelJointState>true</publishWheelJointState>
-        <wheelAcceleration>0.01</wheelAcceleration>
-        <wheelTorque>30</wheelTorque>
+        <wheelAcceleration>10</wheelAcceleration>
+        <wheelTorque>100</wheelTorque>
         <publishTf>1</publishTf>
         <odometrySource>encoder</odometrySource>
         </plugin>
         <!--plugin name="ros_control" filename="libhwi_switch_gazebo_ros_control.so"-->
-        <plugin name="gazebo_ros_control" filename="libgazebo_ros_control.so">
-            <robotNamespace>/mp500lwa4d</robotNamespace>
-            <robotBaseFrame>base_footprint</robotBaseFrame>
-        </plugin>
     </gazebo>
   </robot>

Commit message: Organized files

File: urdf/base/base.gazebo.xacro (robot description, xacro)
@@ -32,8 +32,9 @@
       <gazebo reference="hanger">
           <gravity>true</gravity>
-          <mu1>0.1</mu1>
-          <mu2>0.1</mu2>
+          <mu1>100.5</mu1>
+          <mu2>100.5</mu2>
           <kp>1000000.0</kp>
           <kd>100.0</kd>
+          <fdir1>0 0 1</fdir1>
           <material value="Gazebo/Grey"/>
       </gazebo>

File: urdf/base/base_mp500.urdf.xacro (robot description, xacro)
@@ -18,5 +18,5 @@
 	<link name="base_link">
 		<inertial>
-			<mass value="1" />
+			<mass value="10" />
 			<!--<origin xyz="0 0 0.216" rpy="0 0 0"/>-->
 			<!--<inertia ixx="0.54" ixy="0.0" ixz="0.0" iyy="1.08" iyz="0.0" izz="1.23" />-->
@@ -31,5 +31,5 @@
 				<mesh filename="package://mp500lwa4d_description/meshes/mp500/MP500-BODY.STL" scale="0.01 0.01 0.01"/>
 			<!--cylinder length="0.381" radius="0.2545"/-->
-			<!--box size="0.445 0.277 0.17"/-->
+				<!--<box size="0.445 0.277 0.17"/>-->
 			</geometry>
 			<material name="Grey" />
@@ -38,4 +38,5 @@
 			<origin xyz="0 0 0.216" rpy="0 0 -1.57" />
 			<geometry>
+				<!--<mesh filename="package://mp500lwa4d_description/meshes/mp500/MP500-BODY.STL" scale="0.01 0.01 0.01"/>-->
 				<box size="0.400 0.676 0.300"/>
 				<!--cylinder length="0.381" radius="0.2545"/-->
@@ -135,5 +136,5 @@
 	<link name="hanger">
 		<inertial>
-			<mass value="0.01" />
+			<mass value="1" />
 			<origin xyz="0 0 0" rpy="0 0 0" />
 			<inertia ixx="0.0013" ixy="0" ixz="0" iyy="0.0013" iyz="0" izz="0.0013" />
